File: Clippy.kicad_pcb (KiCad board)
At the start: 2 copper layers, 61.2 x 38.4 mm, 19 parts, among them J1 Conn_01x08, SW1 PEC11R-4215F-S0024, U1 tiny2040, U2 SN74LV1T34DBV

Commit message: Edit schematic labels, initial keymap
Parts:
- SW1: value PEC11R-4215F-S0024 -> PEC12R-4215F-S0024
Connections:
- D1 pad 1: ROW0 -> ROW1
- D2 pad 1: ROW0 -> ROW1
- D3 pad 1: ROW1 -> ROW0
- D4 pad 1: ROW1 -> ROW0
- U1 pad 10: ROW1 -> ROW0
- U1 pad 9: ROW0 -> ROW1
Routing:
- net ROW1: track 19.1 -> 18.1 mm
- net ROW0: track 18.1 -> 19.1 mm
Changed lines of the file:
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@@
       (stroke (width 0.1) (type solid)) (layer "F.Fab"))
     (pad "1" thru_hole rect (at 0 0 315) (size 1.6 1.6) (drill 0.8) (layers "*.Cu" "*.Mask")
-      (net 5 "ROW1") (pinfunction "K") (pintype "passive"))
+      (net 6 "ROW0") (pinfunction "K") (pintype "passive"))
     (pad "2" thru_hole oval (at 7.62 0 315) (size 1.6 1.6) (drill 0.8) (layers "*.Cu" "*.Mask")
       (net 10 "Net-(D3-A)") (pinfunction "A") (pintype "passive"))
@@
       (net 19 "GND") (pinfunction "GND") (pintype "input") (solder_mask_margin 0.1016))
     (pad "9" thru_hole circle (at 16.62 10.132381) (size 1.7526 1.7526) (drill 1.0922) (layers "*.Cu" "*.Mask")
-      (net 6 "ROW0") (pinfunction "GP7") (pintype "input") (solder_mask_margin 0.1016))
+      (net 5 "ROW1") (pinfunction "GP7") (pintype "input") (solder_mask_margin 0.1016))
     (pad "9" smd rect (at 17.4963 10.132381) (size 3.5 1.7526) (layers "F.Cu" "F.Mask")
-      (net 6 "ROW0") (pinfunction "GP7") (pintype "input") (solder_mask_margin 0.1016))
+      (net 5 "ROW1") (pinfunction "GP7") (pintype "input") (solder_mask_margin 0.1016))
     (pad "10" thru_hole circle (at 16.62 7.592381) (size 1.7526 1.7526) (drill 1.0922) (layers "*.Cu" "*.Mask")
-      (net 5 "ROW1") (pinfunction "GP6") (pintype "input") (solder_mask_margin 0.1016))
+      (net 6 "ROW0") (pinfunction "GP6") (pintype "input") (solder_mask_margin 0.1016))
     (pad "10" smd rect (at 17.4963 7.592381) (size 3.5 1.7526) (layers "F.Cu" "F.Mask")
-      (net 5 "ROW1") (pinfunction "GP6") (pintype "input") (solder_mask_margin 0.1016))
+      (net 6 "ROW0") (pinfunction "GP6") (pintype "input") (solder_mask_margin 0.1016))
     (pad "11" thru_hole circle (at 16.62 5.052381) (size 1.7526 1.7526) (drill 1.0922) (layers "*.Cu" "*.Mask")
       (net 20 "ENC1") (pinfunction "GP5") (pintype "input") (solder_mask_margin 0.1016))
@@
       (stroke (width 0.1) (type solid)) (layer "F.Fab"))
     (pad "1" thru_hole rect (at 0 0 315) (size 1.6 1.6) (drill 0.8) (layers "*.Cu" "*.Mask")
-      (net 5 "ROW1") (pinfunction "K") (pintype "passive"))
+      (net 6 "ROW0") (pinfunction "K") (pintype "passive"))
     (pad "2" thru_hole oval (at 7.62 0 315) (size 1.6 1.6) (drill 0.8) (layers "*.Cu" "*.Mask")
       (net 9 "Net-(D4-A)") (pinfunction "A") (pintype "passive"))
@@
       (stroke (width 0.1) (type solid)) (layer "F.Fab"))
     (pad "1" thru_hole rect (at 0 0 315) (size 1.6 1.6) (drill 0.8) (layers "*.Cu" "*.Mask")
-      (net 6 "ROW0") (pinfunction "K") (pintype "passive"))
+      (net 5 "ROW1") (pinfunction "K") (pintype "passive"))
     (pad "2" thru_hole oval (at 7.62 0 315) (size 1.6 1.6) (drill 0.8) (layers "*.Cu" "*.Mask")
       (net 12 "Net-(D1-A)") (pinfunction "A") (pintype "passive"))
@@
       (stroke (width 0.1) (type solid)) (layer "F.Fab"))
     (pad "1" thru_hole rect (at 0 0 315) (size 1.6 1.6) (drill 0.8) (layers "*.Cu" "*.Mask")
-      (net 6 "ROW0") (pinfunction "K") (pintype "passive"))
+      (net 5 "ROW1") (pinfunction "K") (pintype "passive"))
     (pad "2" thru_hole oval (at 7.62 0 315) (size 1.6 1.6) (drill 0.8) (layers "*.Cu" "*.Mask")
       (net 11 "Net-(D2-A)") (pinfunction "A") (pintype "passive"))
@@
         (effects (font (size 1 1) (thickness 0.15)))
     )
-    (fp_text value "PEC11R-4215F-S0024" (at 7.3 11.6 90) (layer "F.Fab")
+    (fp_text value "PEC12R-4215F-S0024" (at 7.3 11.6 90) (layer "F.Fab")
         (effects (font (size 1 1) (thickness 0.15)))
     )
@@
     (fp_arc (start -1.699999 0.702844) (mid -1.712527 0.814069) (end -1.749484 0.919721)
       (stroke (width 0.1) (type solid)) (layer "Edge.Cuts"))
-    (fp_arc (start -1.046711 1.568299) (mid -1.63807 1.504035) (end -1.749484 0.919721)
+    (fp_arc (start -1.046711 1.568299) (mid -1.638071 1.504035) (end -1.749484 0.919721)
       (stroke (width 0.1) (type solid)) (layer "Edge.Cuts"))
     (fp_arc (start -1.046711 1.568299) (mid -0.925123 1.517377) (end -0.794453 1.5)
@@
     (fp_arc (start 1.749484 0.919721) (mid 1.638072 1.504036) (end 1.046711 1.5683)
       (stroke (width 0.1) (type solid)) (layer "Edge.Cuts"))
-    (fp_arc (start 1.749484 0.919721) (mid 1.712534 0.814067) (end 1.699999 0.702843)
+    (fp_arc (start 1.749484 0.919721) (mid 1.71254 0.814067) (end 1.699999 0.702843)
       (stroke (width 0.1) (type solid)) (layer "Edge.Cuts"))
     (fp_line (start -3.8 -1.999999) (end -3.8 2.000001)
@@
     (fp_arc (start -1.699999 0.702844) (mid -1.712527 0.814069) (end -1.749484 0.919721)
       (stroke (width 0.1) (type solid)) (layer "Edge.Cuts"))
-    (fp_arc (start -1.046711 1.568299) (mid -1.63807 1.504035) (end -1.749484 0.919721)
+    (fp_arc (start -1.046711 1.568299) (mid -1.638071 1.504035) (end -1.749484 0.919721)
       (stroke (width 0.1) (type solid)) (layer "Edge.Cuts"))
     (fp_arc (start -1.046711 1.568299) (mid -0.925123 1.517377) (end -0.794453 1.5)
@@
     (fp_arc (start 1.749484 0.919721) (mid 1.638072 1.504036) (end 1.046711 1.5683)
       (stroke (width 0.1) (type solid)) (layer "Edge.Cuts"))
-    (fp_arc (start 1.749484 0.919721) (mid 1.712534 0.814067) (end 1.699999 0.702843)
+    (fp_arc (start 1.749484 0.919721) (mid 1.71254 0.814067) (end 1.699999 0.702843)
       (stroke (width 0.1) (type solid)) (layer "Edge.Cuts"))
     (fp_line (start -3.8 -1.999999) (end -3.8 2.000001)
@@
     (fp_arc (start -1.699999 0.702844) (mid -1.712527 0.814069) (end -1.749484 0.919721)
       (stroke (width 0.1) (type solid)) (layer "Edge.Cuts"))
-    (fp_arc (start -1.046711 1.568299) (mid -1.63807 1.504035) (end -1.749484 0.919721)
+    (fp_arc (start -1.046711 1.568299) (mid -1.638071 1.504035) (end -1.749484 0.919721)
       (stroke (width 0.1) (type solid)) (layer "Edge.Cuts"))
     (fp_arc (start -1.046711 1.568299) (mid -0.925123 1.517377) (end -0.794453 1.5)
@@
     (fp_arc (start 1.749484 0.919721) (mid 1.638072 1.504036) (end 1.046711 1.5683)
       (stroke (width 0.1) (type solid)) (layer "Edge.Cuts"))
-    (fp_arc (start 1.749484 0.919721) (mid 1.712534 0.814067) (end 1.699999 0.702843)
+    (fp_arc (start 1.749484 0.919721) (mid 1.71254 0.814067) (end 1.699999 0.702843)
       (stroke (width 0.1) (type solid)) (layer "Edge.Cuts"))
     (fp_line (start -3.8 -1.999999) (end -3.8 2.000001)
@@
     (effects (font (size 0.75 0.75) (thickness 0.1875) bold) (justify bottom mirror))
   )
-  (segment (start 142.059686 80.518) (end 138.860962 83.716724) (width 0.35) (layer "F.Cu") (net 5))
-  (segment (start 145.26 76.29605) (end 146.685 77.72105) (width 0.35) (layer "F.Cu") (net 5))
-  (segment (start 146.685 79.91365) (end 146.08065 80.518) (width 0.35) (layer "F.Cu") (net 5))
-  (segment (start 146.685 77.72105) (end 146.685 79.91365) (width 0.35) (layer "F.Cu") (net 5))
-  (segment (start 143.51 76.29605) (end 145.26 76.29605) (width 0.35) (layer "F.Cu") (net 5))
-  (segment (start 146.08065 80.518) (end 142.059686 80.518) (width 0.35) (layer "F.Cu") (net 5))
-  (segment (start 135.101763 83.716724) (end 138.860962 83.716724) (width 0.35) (layer "B.Cu") (net 5))
-  (segment (start 131.313809 83.716724) (end 133.039333 81.9912) (width 0.35) (layer "F.Cu") (net 6))
-  (segment (start 141.831869 79.968) (end 142.5868 79.968) (width 0.35) (layer "F.Cu") (net 6))
-  (segment (start 139.808669 81.9912) (end 141.831869 79.968) (width 0.35) (layer "F.Cu") (net 6))
-  (segment (start 143.51 79.0448) (end 143.51 78.83605) (width 0.35) (layer "F.Cu") (net 6))
-  (segment (start 133.039333 81.9912) (end 139.808669 81.9912) (width 0.35) (layer "F.Cu") (net 6))
-  (segment (start 142.5868 79.968) (end 143.51 79.0448) (width 0.35) (layer "F.Cu") (net 6))
-  (segment (start 127.530886 83.716724) (end 131.313809 83.716724) (width 0.35) (layer "B.Cu") (net 6))
+  (segment (start 131.313809 83.716724) (end 133.039333 81.9912) (width 0.35) (layer "F.Cu") (net 5))
+  (segment (start 141.831869 79.968) (end 142.5868 79.968) (width 0.35) (layer "F.Cu") (net 5))
+  (segment (start 139.808669 81.9912) (end 141.831869 79.968) (width 0.35) (layer "F.Cu") (net 5))
+  (segment (start 143.51 79.0448) (end 143.51 78.83605) (width 0.35) (layer "F.Cu") (net 5))
+  (segment (start 133.039333 81.9912) (end 139.808669 81.9912) (width 0.35) (layer "F.Cu") (net 5))
+  (segment (start 142.5868 79.968) (end 143.51 79.0448) (width 0.35) (layer "F.Cu") (net 5))
+  (segment (start 127.530886 83.716724) (end 131.313809 83.716724) (width 0.35) (layer "B.Cu") (net 5))
+  (segment (start 142.059686 80.518) (end 138.860962 83.716724) (width 0.35) (layer "F.Cu") (net 6))
+  (segment (start 145.26 76.29605) (end 146.685 77.72105) (width 0.35) (layer "F.Cu") (net 6))
+  (segment (start 146.685 79.91365) (end 146.08065 80.518) (width 0.35) (layer "F.Cu") (net 6))
+  (segment (start 146.685 77.72105) (end 146.685 79.91365) (width 0.35) (layer "F.Cu") (net 6))
+  (segment (start 143.51 76.29605) (end 145.26 76.29605) (width 0.35) (layer "F.Cu") (net 6))
+  (segment (start 146.08065 80.518) (end 142.059686 80.518) (width 0.35) (layer "F.Cu") (net 6))
+  (segment (start 135.101763 83.716724) (end 138.860962 83.716724) (width 0.35) (layer "B.Cu") (net 6))
   (segment (start 175.365187 90.17) (end 166.624 90.17) (width 0.35) (layer "B.Cu") (net 7))
   (segment (start 166.624 90.17) (end 162.169 94.625) (width 0.35) (layer "B.Cu") (net 7))
